Commit message: converted most of the initial urdf to xacros and generated the two wheels

File: urdf/udacity_bot.xacro (robot description, xacro)
@@ -1,57 +1,131 @@
 <?xml version='1.0'?>
 <robot name="udacity_bot" xmlns:xacro="http://www.ros.org/wiki/xacro">
+ <!-- ################### XACRO Definitions ############################# -->
+ <!-- ################### XACRO Definitions ############################# -->
+ <!-- ################### XACRO Definitions ############################# -->
+ <!-- ################### XACRO Definitions ############################# -->
+ <xacro:macro name="zero_origin">
+     <origin xyz="0 0 0" rpy="0 0 0" />
+ </xacro:macro>
+<xacro:macro name="wheel_link_origin">
+    <origin xyz="0 0 0" rpy="0 1.5707 1.5707" />
+</xacro:macro>
+<xacro:macro name="default_inertia">
+    <inertia
+        ixx="0.1" ixy="0" ixz="0"
+        iyy="0.1" iyz="0"
+        izz="0.1"
+      />
+</xacro:macro>
+<!-- ################### MACRO Generators ############################# -->
+<!-- ################### MACRO Generators ############################# -->
+<!-- ################### MACRO Generators ############################# -->
+<!-- ################### MACRO Generators ############################# -->
+<xacro:macro name="generate_geometry" params="shape radius=0 length=0 x=0 y=0 z=0">
+<!--UNITS IN METERS-->
+<!--<cylinder radius="" length=""/>-->
+<!--<box x="" y="" z="" />-->
+<!--<sphere radius=""/> -->
+    <geometry>
+        <xacro:if value="${shape == 'box'}">
+            <box size="${x} ${y} ${z}"/>
+        </xacro:if>
+        <xacro:if value="${shape == 'cylinder'}">
+            <cylinder length="${length}" radius="${radius}"/>
+        </xacro:if>
+        <xacro:if value="${shape == 'sphere'}">
+            <sphere radius="${radius}"/>
+        </xacro:if>
+    </geometry>
+</xacro:macro>
+<xacro:macro name="generate_wheel_link" params="side">
+    <link name="${side}_wheel">
+       <inertial>
+           <xacro:wheel_link_origin/>
+           <mass value="5"/>
+           <xacro:default_inertia/>
+       </inertial>
+       <collision>
+             <xacro:wheel_link_origin/>
+             <xacro:generate_geometry shape="cylinder" radius="0.1" length="0.05" />
+       </collision>
+       <visual>
+             <xacro:wheel_link_origin/>
+             <xacro:generate_geometry shape="cylinder" radius="0.1" length="0.05" />
+       </visual>
+   </link>
+</xacro:macro>
+<xacro:macro name="generate_wheel_joint" params="side">
+    <joint type="continuous" name="${side}_wheel_hinge">
+        <xacro:if value="${side == 'left'}">
+            <origin xyz="0 0.15 0" rpy="0 0 0"/>
+        </xacro:if>
+        <xacro:if value="${side == 'right'}">
+            <origin xyz="0 -0.15 0" rpy="0 0 0"/>
+        </xacro:if>
+        <parent link="chassis"/>
+        <child link="${side}_wheel"/>
+        <axis xyz="0 1 0" rpy="0 0 0"/>
+        <limit effort="10000" velocity="1000"/>
+        <dynamics damping="1.0" friction="1.0"/>
+    </joint>
+</xacro:macro>
+ <!-- ################### ROBOT Definitions ############################# -->
+ <!-- ################### ROBOT Definitions ############################# -->
+ <!-- ################### ROBOT Definitions ############################# -->
+ <!-- ################### ROBOT Definitions ############################# -->
   <link name="robot_footprint"></link>
   <joint name="robot_footprint_joint" type="fixed">
-    <origin xyz="0 0 0" rpy="0 0 0" />
-    <parent link="robot_footprint"/>
-    <child link="chassis" />
+      <origin xyz="0 0 0" rpy="0 0 0" />
+      <parent link="robot_footprint"/>
+      <child link="chassis" />
   </joint>
   <link name='chassis'>
-    <pose>0 0 0.1 0 0 0</pose>
-    <inertial>
-      <mass value="15.0"/>
-      <origin xyz="0.0 0 0" rpy=" 0 0 0"/>
-      <inertia
-          ixx="0.1" ixy="0" ixz="0"
-          iyy="0.1" iyz="0"
-          izz="0.1"
-      />
+      <pose>0 0 0.1 0 0 0</pose>
+      <inertial>
+          <mass value="15.0"/>
+          <origin xyz="0.0 0 0" rpy=" 0 0 0"/>
+          <xacro:default_inertia/>
     </inertial>
     <collision name='collision'>
-      <origin xyz="0 0 0" rpy=" 0 0 0"/>
-      <geometry>
-        <box size=".4 .2 .1"/>
-      </geometry>
+        <xacro:zero_origin/>
+        <geometry>
+            <box size=".4 .2 .1"/>
+        </geometry>
     </collision>
     <visual name='chassis_visual'>
-      <origin xyz="0 0 0" rpy=" 0 0 0"/>
-      <geometry>
-        <box size=".4 .2 .1"/>
-      </geometry>
+        <xacro:zero_origin/>
+        <geometry>
+            <box size=".4 .2 .1"/>
+        </geometry>
     </visual>
     <collision name='back_caster_collision'>
-      <origin xyz="-0.15 0 -0.05" rpy=" 0 0 0"/>
-      <geometry>
-        <sphere radius="0.0499"/>
-      </geometry>
+        <origin xyz="-0.15 0 -0.05" rpy=" 0 0 0"/>
+        <geometry>
+            <sphere radius="0.0499"/>
+        </geometry>
     </collision>
     <visual name='back_caster_visual'>
-      <origin xyz="-0.15 0 -0.05" rpy=" 0 0 0"/>
-      <geometry>
-        <sphere radius="0.05"/>
-      </geometry>
+        <origin xyz="-0.15 0 -0.05" rpy=" 0 0 0"/>
+        <geometry>
+            <sphere radius="0.05"/>
+        </geometry>
     </visual>
     <collision name='front_caster_collision'>
-      <origin xyz="0.15 0 -0.05" rpy=" 0 0 0"/>
-      <geometry>
-        <sphere radius="0.0499"/>
-      </geometry>
+        <origin xyz="0.15 0 -0.05" rpy=" 0 0 0"/>
+        <geometry>
+            <sphere radius="0.0499"/>
+        </geometry>
     </collision>
     <visual name='front_caster_visual'>
-      <origin xyz="0.15 0 -0.05" rpy=" 0 0 0"/>
-      <geometry>
-        <sphere radius="0.05"/>
-      </geometry>
+        <origin xyz="0.15 0 -0.05" rpy=" 0 0 0"/>
+        <geometry>
+            <sphere radius="0.05"/>
+        </geometry>
     </visual>
   </link>
+  <xacro:generate_wheel_link side="right"/>
+  <xacro:generate_wheel_link side="left"/>
+  <xacro:generate_wheel_joint side="right"/>
+  <xacro:generate_wheel_joint side="left"/>
 </robot>

Commit message: adding hokuya laser

File: urdf/udacity_bot.xacro (robot description, xacro)
@@ -1,8 +1,10 @@
 <?xml version='1.0'?>
 <robot name="udacity_bot" xmlns:xacro="http://www.ros.org/wiki/xacro">
- <!-- ################### XACRO Definitions ############################# -->
- <!-- ################### XACRO Definitions ############################# -->
- <!-- ################### XACRO Definitions ############################# -->
- <!-- ################### XACRO Definitions ############################# -->
+<!-- ################### XACRO Definitions ############################# -->
+<!-- ################### XACRO Definitions ############################# -->
+<!-- ################### XACRO Definitions ############################# -->
+<!-- ################### XACRO Definitions ############################# -->
+<xacro:property name="min_mass" value="0.1"/>
+<!-- ################### XACRO Origins ############################# -->
  <xacro:macro name="zero_origin">
      <origin xyz="0 0 0" rpy="0 0 0" />
@@ -11,4 +13,5 @@
     <origin xyz="0 0 0" rpy="0 1.5707 1.5707" />
 </xacro:macro>
+<!-- ################### XACRO Inertias ############################# -->
 <xacro:macro name="default_inertia">
     <inertia
@@ -16,4 +19,11 @@
         iyy="0.1" iyz="0"
         izz="0.1"
+      />
+</xacro:macro>
+<xacro:macro name="min_inertia">
+    <inertia
+        ixx="1e-6" ixy="0" ixz="0"
+        iyy="1e-6" iyz="0"
+        izz="1e-6"
       />
 </xacro:macro>
@@ -75,5 +85,5 @@
  <!-- ################### ROBOT Definitions ############################# -->
  <!-- ################### ROBOT Definitions ############################# -->
-  <link name="robot_footprint"></link>
+<link name="robot_footprint"></link>
   <joint name="robot_footprint_joint" type="fixed">
       <origin xyz="0 0 0" rpy="0 0 0" />
@@ -81,4 +91,5 @@
       <child link="chassis" />
   </joint>
+<!-- BEGIN Chassis -->
   <link name='chassis'>
       <pose>0 0 0.1 0 0 0</pose>
@@ -124,8 +135,33 @@
         </geometry>
     </visual>
-  </link>
-  <xacro:generate_wheel_link side="right"/>
-  <xacro:generate_wheel_link side="left"/>
-  <xacro:generate_wheel_joint side="right"/>
-  <xacro:generate_wheel_joint side="left"/>
+</link>
+<!-- END Chassis -->
+<!-- ################### LINK Definitions ############################# -->
+<!-- ################### LINK Definitions ############################# -->
+<!-- ################### LINK Definitions ############################# -->
+<!-- ################### LINK Definitions ############################# -->
+    <xacro:generate_wheel_link side="right"/>
+    <xacro:generate_wheel_link side="left"/>
+<!-- ################### JOINT Definitions ############################# -->
+<!-- ################### JOINT Definitions ############################# -->
+<!-- ################### JOINT Definitions ############################# -->
+<!-- ################### JOINT Definitions ############################# -->
+    <xacro:generate_wheel_joint side="right"/>
+    <xacro:generate_wheel_joint side="left"/>
+<!-- ################### SENSOR Definitions ############################# -->
+    <link name="camera">
+        <inertial>
+            <xacro:zero_origin/>
+            <mass value="${min_mass}"/>
+            <xacro:min_inertia/>
+        </inertial>
+        <collision>
+            <xacro:zero_origin/>
+            <xacro:generate_geometry shape="box" x="0.05" y="0.05" z="0.05"/>
+        </collision>
+        <visual>
+            <xacro:zero_origin/>
+            <xacro:generate_geometry shape="box" x="0.05" y="0.05" z="0.05"/>
+        </visual>
+    </link>
 </robot>

Commit message: mesh is visible in rviz, but not in gazebo. tried another dae mesh and it behaves the same way. gonna try in diff workspace

File: urdf/udacity_bot.xacro (robot description, xacro)
@@ -149,10 +149,16 @@
     <xacro:generate_wheel_joint side="right"/>
     <xacro:generate_wheel_joint side="left"/>
-<!-- ################### SENSOR Definitions ############################# -->
-    <link name="camera">
+    <joint name="camera_joint" type="fixed">
+        <origin xyz="0.2 0 0" rpy="0 0 0"/>
+        <parent link="chassis"/>
+        <child link="camera_link"/>
+    </joint>
+ <!--################### SENSOR Definitions ############################# -->
+    <link name="camera_link">
         <inertial>
             <xacro:zero_origin/>
-            <mass value="${min_mass}"/>
-            <xacro:min_inertia/>
+            <!--<mass value="${min_mass}"/>-->
+            <mass value="0.1"/>
+            <xacro:default_inertia/>
         </inertial>
         <collision>
@@ -165,3 +171,34 @@
         </visual>
     </link>
+    <link name="hokuyo_link">
+        <inertial>
+            <xacro:zero_origin/>
+            <!--<mass value="${min_mass}"/>-->
+            <mass value="0.1"/>
+            <xacro:default_inertia/>
+        </inertial>
+        <collision>
+            <xacro:zero_origin/>
+            <xacro:generate_geometry shape="box" x="0.1" y="0.1" z="0.1"/>
+        </collision>
+        <visual>
+            <xacro:zero_origin/>
+            <!--<xacro:generate_geometry shape="box" x="0.05" y="0.05" z="0.05"/>-->
+            <geometry>
+                <mesh filename="package://udacity_bot/models/meshes/hokuyo.dae"/>
+            </geometry>
+        </visual>
+    </link>
+    <joint name="hokuyo_joint" type="fixed">
+        <origin xyz="0.15 0 0.1" rpy="0 0 0"/>
+        <parent link="chassis"/>
+        <child link="hokuyo_link"/>
+    </joint>
+    <gazebo reference="hokuyo_link">
+        <kp>1000.0</kp>
+        <kd>1000.0</kd>
+        <mu1>10.0</mu1>
+        <mu2>10.0</mu2>
+        <material>Gazebo/Green</material>
+        </gazebo>
 </robot>

Commit message: gazebo world giving me an error about having two identical packages?

File: urdf/udacity_bot.xacro (robot description, xacro)
@@ -1,4 +1,6 @@
 <?xml version='1.0'?>
 <robot name="udacity_bot" xmlns:xacro="http://www.ros.org/wiki/xacro">
+<!--Includes Sensor Plugins defined in .gazebo file-->
+<!--<xacro:include filename="$(find udacity_bot)/urdf/udacity_bot.gazebo" />-->
 <!-- ################### XACRO Definitions ############################# -->
 <!-- ################### XACRO Definitions ############################# -->
@@ -32,4 +34,13 @@
 <!-- ################### MACRO Generators ############################# -->
 <!-- ################### MACRO Generators ############################# -->
+<xacro:macro name="generate_gazebo_reference" params="link_name color">
+    <gazebo reference="${link_name}">
+        <!--<kp>1000.0</kp>-->
+        <!--<kd>1000.0</kd>-->
+        <!--<mu1>10.0</mu1>-->
+        <!--<mu2>10.0</mu2>-->
+        <material>Gazebo/${color}</material>
+    </gazebo>
+</xacro:macro>
 <xacro:macro name="generate_geometry" params="shape radius=0 length=0 x=0 y=0 z=0">
 <!--UNITS IN METERS-->
@@ -65,4 +76,5 @@
        </visual>
    </link>
+   <xacro:generate_gazebo_reference link_name="${side}_wheel" color="Red"/>
 </xacro:macro>
 <xacro:macro name="generate_wheel_joint" params="side">
@@ -201,4 +213,4 @@
         <mu2>10.0</mu2>
         <material>Gazebo/Green</material>
-        </gazebo>
+    </gazebo>
 </robot>

Commit message: everything is back up and running smoothly. just confirmed laserscan and camera visuals in rviz! and had some fun driving around with my keyboard. next is adding the map

File: urdf/udacity_bot.xacro (robot description, xacro)
@@ -2,5 +2,5 @@
 <robot name="udacity_bot" xmlns:xacro="http://www.ros.org/wiki/xacro">
 <!--Includes Sensor Plugins defined in .gazebo file-->
-<!--<xacro:include filename="$(find udacity_bot)/urdf/udacity_bot.gazebo" />-->
+<xacro:include filename="$(find udacity_bot)/urdf/udacity_bot.gazebo" />
 <!-- ################### XACRO Definitions ############################# -->
 <!-- ################### XACRO Definitions ############################# -->
@@ -76,5 +76,5 @@
        </visual>
    </link>
-   <xacro:generate_gazebo_reference link_name="${side}_wheel" color="Red"/>
+   <xacro:generate_gazebo_reference link_name="${side}_wheel" color="Green"/>
 </xacro:macro>
 <xacro:macro name="generate_wheel_joint" params="side">
@@ -161,4 +161,21 @@
     <xacro:generate_wheel_joint side="right"/>
     <xacro:generate_wheel_joint side="left"/>
+ <!--################### SENSOR Definitions ############################# -->
+    <link name="camera_link">
+        <inertial>
+            <xacro:zero_origin/>
+            <!--<mass value="${min_mass}"/>-->
+            <mass value="0.1"/>
+            <xacro:default_inertia/>
+        </inertial>
+        <collision>
+            <xacro:zero_origin/>
+            <xacro:generate_geometry shape="box" x="0.05" y="0.05" z="0.05"/>
+        </collision>
+        <visual>
+            <xacro:zero_origin/>
+            <xacro:generate_geometry shape="box" x="0.05" y="0.05" z="0.05"/>
+        </visual>
+    </link>
     <joint name="camera_joint" type="fixed">
         <origin xyz="0.2 0 0" rpy="0 0 0"/>
@@ -166,21 +183,4 @@
         <child link="camera_link"/>
     </joint>
- <!--################### SENSOR Definitions ############################# -->
-    <link name="camera_link">
-        <inertial>
-            <xacro:zero_origin/>
-            <!--<mass value="${min_mass}"/>-->
-            <mass value="0.1"/>
-            <xacro:default_inertia/>
-        </inertial>
-        <collision>
-            <xacro:zero_origin/>
-            <xacro:generate_geometry shape="box" x="0.05" y="0.05" z="0.05"/>
-        </collision>
-        <visual>
-            <xacro:zero_origin/>
-            <xacro:generate_geometry shape="box" x="0.05" y="0.05" z="0.05"/>
-        </visual>
-    </link>
     <link name="hokuyo_link">
         <inertial>
@@ -207,10 +207,3 @@
         <child link="hokuyo_link"/>
     </joint>
-    <gazebo reference="hokuyo_link">
-        <kp>1000.0</kp>
-        <kd>1000.0</kd>
-        <mu1>10.0</mu1>
-        <mu2>10.0</mu2>
-        <material>Gazebo/Green</material>
-    </gazebo>
 </robot>

Commit message: started testing out parameters. in general, the bot is able to correctly generate a global plan, but chooses really weird local paths. it tends to take corners very very very widely.

File: urdf/udacity_bot.xacro (robot description, xacro)
@@ -162,5 +162,5 @@
     <xacro:generate_wheel_joint side="left"/>
  <!--################### SENSOR Definitions ############################# -->
-    <link name="camera_link">
+    <link name="camera">
         <inertial>
             <xacro:zero_origin/>
@@ -181,7 +181,7 @@
         <origin xyz="0.2 0 0" rpy="0 0 0"/>
         <parent link="chassis"/>
-        <child link="camera_link"/>
+        <child link="camera"/>
     </joint>
-    <link name="hokuyo_link">
+    <link name="hokuyo">
         <inertial>
             <xacro:zero_origin/>
@@ -205,5 +205,5 @@
         <origin xyz="0.15 0 0.1" rpy="0 0 0"/>
         <parent link="chassis"/>
-        <child link="hokuyo_link"/>
+        <child link="hokuyo"/>
     </joint>
 </robot>

Commit message: commented out each param file to the classroom code, and one or two unmentioned params

File: urdf/udacity_bot.xacro (robot description, xacro)
@@ -34,8 +34,8 @@
 <xacro:macro name="generate_gazebo_reference" params="link_name color">
     <gazebo reference="${link_name}">
-        <kp>10000000.0</kp>
+        <!-- <kp>10000000.0</kp>
         <kd>1.0</kd>
         <mu1>1.0</mu1>
-        <mu2>1.0</mu2>
+        <mu2>1.0</mu2> -->
         <material>Gazebo/${color}</material>
     </gazebo>
@@ -88,5 +88,5 @@
         <axis xyz="0 1 0" rpy="0 0 0"/>
         <limit effort="10000" velocity="1000"/>
-        <dynamics damping="1.0" friction="1.0"/>
+        <joint_properties damping="1.0" friction="1.0"/>
     </joint>
 </xacro:macro>
@@ -126,5 +126,5 @@
         <origin xyz="-0.15 0 -0.05" rpy=" 0 0 0"/>
         <geometry>
-            <sphere radius="0.0499"/>
+            <sphere radius="0.05"/>
         </geometry>
         <surface>

Commit message: testing out shell

File: urdf/udacity_bot.xacro (robot description, xacro)
@@ -7,4 +7,7 @@
 <xacro:property name="min_mass" value="0.1"/>
 <!-- ################### XACRO Origins ############################# -->
+ <xacro:macro name="shell_origin">
+     <origin xyz="0 0 -.085" rpy="0 -0.1 3.14159" />
+ </xacro:macro>
  <xacro:macro name="zero_origin">
      <origin xyz="0 0 0" rpy="0 0 0" />
@@ -105,5 +108,5 @@
 <!-- BEGIN Chassis -->
   <link name='chassis'>
-      <pose>0 0 0.1 0 0 0</pose>
+      <pose>0 0 0 0 0 0</pose>
       <inertial>
           <mass value="15.0"/>
@@ -118,7 +121,9 @@
     </collision>
     <visual name='chassis_visual'>
-        <xacro:zero_origin/>
-        <geometry>
-            <box size=".4 .2 .1"/>
+        <!-- <xacro:zero_origin/> -->
+        <xacro:shell_origin/>
+        <geometry>
+            <!-- <box size=".4 .2 .1"/> -->
+            <mesh filename="package://udacity_bot/models/meshes/green_shell.dae"/>
         </geometry>
     </visual>
