Commit message: shell fits

File: urdf/shell.xacro (robot description, xacro)
@@ -121,7 +121,9 @@
     </collision>
     <visual name='chassis_visual'>
-        <xacro:zero_origin/>
-        <geometry>
-            <box size=".4 .2 .1"/>
+        <!-- <xacro:zero_origin/> -->
+        <xacro:shell_origin/>
+        <geometry>
+            <!-- <box size=".4 .2 .1"/> -->
+            <mesh filename="package://udacity_bot/models/meshes/green_shell.dae"/>
         </geometry>
     </visual>

Commit message: edited locations of shell components

File: urdf/shell.xacro (robot description, xacro)
@@ -117,5 +117,6 @@
         <xacro:zero_origin/>
         <geometry>
-            <box size=".4 .2 .1"/>
+            <!-- <box size=".4 .2 .1"/> -->
+            <sphere radius="0.15"/>
         </geometry>
     </collision>
@@ -129,7 +130,7 @@
     </visual>
     <collision name='back_caster_collision'>
-        <origin xyz="-0.15 0 -0.05" rpy=" 0 0 0"/>
-        <geometry>
-            <sphere radius="0.05"/>
+        <origin xyz="-0.1 0 -0.02" rpy=" 0 0 0"/>
+        <geometry>
+            <sphere radius="0.01"/>
         </geometry>
         <surface>
@@ -145,10 +146,10 @@
     </collision>
     <visual name='back_caster_visual'>
-        <origin xyz="-0.15 0 -0.05" rpy=" 0 0 0"/>
-        <geometry>
-            <sphere radius="0.05"/>
+        <origin xyz="-0.1 0 -0.02" rpy=" 0 0 0"/>
+        <geometry>
+            <sphere radius="0.01"/>
         </geometry>
     </visual>
-    <collision name='front_caster_collision'>
+    <!-- <collision name='front_caster_collision'>
         <origin xyz="0.15 0 -0.05" rpy=" 0 0 0"/>
         <geometry>
@@ -172,5 +173,5 @@
         </geometry>
     </visual>
-</link>
+</link> -->
 <!-- END Chassis -->
 <!-- ################### LINK Definitions ############################# -->
@@ -228,5 +229,5 @@
     </link>
     <joint name="hokuyo_joint" type="fixed">
-        <origin xyz="0.15 0 0.1" rpy="0 0 0"/>
+        <origin xyz="0.13 0 0.13" rpy="0 0 0"/>
         <parent link="chassis"/>
         <child link="hokuyo"/>

Commit message: shell_bot (aka shelly) is now a functional vehicle. next is to tune her params!

File: urdf/shell.xacro (robot description, xacro)
@@ -9,4 +9,7 @@
  <xacro:macro name="shell_origin">
      <origin xyz="0 0 -.1" rpy="-.1 0 1.5707" />
+ </xacro:macro>
+  <xacro:macro name="shell_collision_origin">
+     <origin xyz="0 0 -.1" rpy="0 0 0" />
  </xacro:macro>
  <xacro:macro name="zero_origin">
@@ -77,13 +80,13 @@
        </visual>
    </link>
-   <xacro:generate_gazebo_reference link_name="${side}_wheel" color="Green"/>
+   <xacro:generate_gazebo_reference link_name="${side}_wheel" color="GreyTransparent"/>
 </xacro:macro>
 <xacro:macro name="generate_wheel_joint" params="side">
     <joint type="continuous" name="${side}_wheel_hinge">
         <xacro:if value="${side == 'left'}">
-            <origin xyz="0 0.15 0" rpy="0 0 0"/>
+            <origin xyz="0.1 0.169 0" rpy="0 0 0"/>
         </xacro:if>
         <xacro:if value="${side == 'right'}">
-            <origin xyz="0 -0.15 0" rpy="0 0 0"/>
+            <origin xyz="0.1 -0.169 0" rpy="0 0 0"/>
         </xacro:if>
         <parent link="chassis"/>
@@ -115,8 +118,9 @@
     </inertial>
     <collision name='collision'>
-        <xacro:zero_origin/>
+        <xacro:shell_origin/>
         <geometry>
             <!-- <box size=".4 .2 .1"/> -->
-            <sphere radius="0.15"/>
+            <!--<sphere radius="0.01"/>-->
+            <mesh filename="package://udacity_bot/models/meshes/green_shell.dae"/>
         </geometry>
     </collision>
@@ -127,4 +131,14 @@
             <!-- <box size=".4 .2 .1"/> -->
             <mesh filename="package://udacity_bot/models/meshes/green_shell.dae"/>
+            <surface>
+              <friction>
+                    <ode>
+                        <mu>0</mu>
+                        <mu2>0</mu2>
+                        <slip1>1.0</slip1>
+                        <slip2>1.0</slip2>
+                    </ode>
+              </friction>
+        </surface>
         </geometry>
     </visual>
@@ -173,5 +187,6 @@
         </geometry>
     </visual>
-</link> -->
+    -->
+</link>
 <!-- END Chassis -->
 <!-- ################### LINK Definitions ############################# -->
@@ -197,13 +212,14 @@
         <collision>
             <xacro:zero_origin/>
-            <xacro:generate_geometry shape="box" x="0.05" y="0.05" z="0.05"/>
+            <xacro:generate_geometry shape="sphere" radius="0.02"/>
         </collision>
         <visual>
             <xacro:zero_origin/>
-            <xacro:generate_geometry shape="box" x="0.05" y="0.05" z="0.05"/>
+            <xacro:generate_geometry shape="sphere" radius="0.01"/>
         </visual>
     </link>
+    <xacro:generate_gazebo_reference link_name="camera" color="Red"/>
     <joint name="camera_joint" type="fixed">
-        <origin xyz="0.2 0 0" rpy="0 0 0"/>
+        <origin xyz="0.1 0 0" rpy="0 0 0"/>
         <parent link="chassis"/>
         <child link="camera"/>
@@ -229,5 +245,5 @@
     </link>
     <joint name="hokuyo_joint" type="fixed">
-        <origin xyz="0.13 0 0.13" rpy="0 0 0"/>
+        <origin xyz="-0.02 0 0.153" rpy="0 0 0"/>
         <parent link="chassis"/>
         <child link="hokuyo"/>

Commit message: testing stability of shell chassis

File: urdf/shell.xacro (robot description, xacro)
@@ -118,27 +118,17 @@
     </inertial>
     <collision name='collision'>
-        <xacro:shell_origin/>
-        <geometry>
-            <!-- <box size=".4 .2 .1"/> -->
+        <xacro:zero_origin/>
+        <geometry>
+            <box size=".4 .2 .1"/>
             <!--<sphere radius="0.01"/>-->
-            <mesh filename="package://udacity_bot/models/meshes/green_shell.dae"/>
+            <!-- <mesh filename="package://udacity_bot/models/meshes/green_shell.dae"/> -->
         </geometry>
     </collision>
     <visual name='chassis_visual'>
         <!-- <xacro:zero_origin/> -->
-        <xacro:shell_origin/>
+        <xacro:zero_origin/>
         <geometry>
             <!-- <box size=".4 .2 .1"/> -->
             <mesh filename="package://udacity_bot/models/meshes/green_shell.dae"/>
-            <surface>
-              <friction>
-                    <ode>
-                        <mu>0</mu>
-                        <mu2>0</mu2>
-                        <slip1>1.0</slip1>
-                        <slip2>1.0</slip2>
-                    </ode>
-              </friction>
-        </surface>
         </geometry>
     </visual>
@@ -165,5 +155,5 @@
         </geometry>
     </visual>
-    <!-- <collision name='front_caster_collision'>
+    <collision name='front_caster_collision'>
         <origin xyz="0.15 0 -0.05" rpy=" 0 0 0"/>
         <geometry>
@@ -187,5 +177,4 @@
         </geometry>
     </visual>
-    -->
 </link>
 <!-- END Chassis -->

Commit message: shelly is now officially an autonomous, levitating green koopa troopa shell

File: urdf/shell.xacro (robot description, xacro)
@@ -8,8 +8,5 @@
 <!-- ################### XACRO Origins ############################# -->
  <xacro:macro name="shell_origin">
-     <origin xyz="0 0 -.1" rpy="-.1 0 1.5707" />
- </xacro:macro>
-  <xacro:macro name="shell_collision_origin">
-     <origin xyz="0 0 -.1" rpy="0 0 0" />
+     <origin xyz="0 0 0" rpy="0 0 -1.5707" />
  </xacro:macro>
  <xacro:macro name="zero_origin">
@@ -77,16 +74,17 @@
        <visual>
              <xacro:wheel_link_origin/>
-             <xacro:generate_geometry shape="cylinder" radius="0.1" length="0.05" />
+             <!--<xacro:generate_geometry shape="cylinder" radius="0.1" length="0.05" />-->
+             <xacro:generate_geometry shape="sphere" radius="0.001"/>
        </visual>
    </link>
-   <xacro:generate_gazebo_reference link_name="${side}_wheel" color="GreyTransparent"/>
+   <!--<xacro:generate_gazebo_reference link_name="${side}_wheel" color="Green"/>-->
 </xacro:macro>
 <xacro:macro name="generate_wheel_joint" params="side">
     <joint type="continuous" name="${side}_wheel_hinge">
         <xacro:if value="${side == 'left'}">
-            <origin xyz="0.1 0.169 0" rpy="0 0 0"/>
+            <origin xyz="0 0.15 0" rpy="0 0 0"/>
         </xacro:if>
         <xacro:if value="${side == 'right'}">
-            <origin xyz="0.1 -0.169 0" rpy="0 0 0"/>
+            <origin xyz="0 -0.15 0" rpy="0 0 0"/>
         </xacro:if>
         <parent link="chassis"/>
@@ -121,20 +119,18 @@
         <geometry>
             <box size=".4 .2 .1"/>
-            <!--<sphere radius="0.01"/>-->
-            <!-- <mesh filename="package://udacity_bot/models/meshes/green_shell.dae"/> -->
         </geometry>
     </collision>
     <visual name='chassis_visual'>
-        <!-- <xacro:zero_origin/> -->
-        <xacro:zero_origin/>
-        <geometry>
-            <!-- <box size=".4 .2 .1"/> -->
+        <!--<xacro:zero_origin/>-->
+        <xacro:shell_origin/>
+        <geometry>
+            <!--<box size=".4 .2 .1"/> -->
             <mesh filename="package://udacity_bot/models/meshes/green_shell.dae"/>
         </geometry>
     </visual>
     <collision name='back_caster_collision'>
-        <origin xyz="-0.1 0 -0.02" rpy=" 0 0 0"/>
-        <geometry>
-            <sphere radius="0.01"/>
+        <origin xyz="-0.15 0 -0.05" rpy=" 0 0 0"/>
+        <geometry>
+            <sphere radius="0.0499"/>
         </geometry>
         <surface>
@@ -150,7 +146,7 @@
     </collision>
     <visual name='back_caster_visual'>
-        <origin xyz="-0.1 0 -0.02" rpy=" 0 0 0"/>
-        <geometry>
-            <sphere radius="0.01"/>
+        <origin xyz="-0.15 0 -0.05" rpy=" 0 0 0"/>
+        <geometry>
+            <sphere radius="0.001"/>
         </geometry>
     </visual>
@@ -174,5 +170,5 @@
         <origin xyz="0.15 0 -0.05" rpy=" 0 0 0"/>
         <geometry>
-            <sphere radius="0.05"/>
+            <sphere radius="0.001"/>
         </geometry>
     </visual>
@@ -201,14 +197,14 @@
         <collision>
             <xacro:zero_origin/>
-            <xacro:generate_geometry shape="sphere" radius="0.02"/>
+            <xacro:generate_geometry shape="box" x="0.05" y="0.05" z="0.05"/>
         </collision>
         <visual>
             <xacro:zero_origin/>
-            <xacro:generate_geometry shape="sphere" radius="0.01"/>
+            <!--<xacro:generate_geometry shape="box" x="0.05" y="0.05" z="0.05"/>-->
+            <xacro:generate_geometry shape="sphere" radius="0.001"/>
         </visual>
     </link>
-    <xacro:generate_gazebo_reference link_name="camera" color="Red"/>
     <joint name="camera_joint" type="fixed">
-        <origin xyz="0.1 0 0" rpy="0 0 0"/>
+        <origin xyz="0.2 0 0" rpy="0 0 0"/>
         <parent link="chassis"/>
         <child link="camera"/>
@@ -227,12 +223,14 @@
         <visual>
             <xacro:zero_origin/>
-            <!--<xacro:generate_geometry shape="box" x="0.05" y="0.05" z="0.05"/>-->
+            <xacro:generate_geometry shape="sphere" radius="0.001"/>
+            <!--
             <geometry>
                 <mesh filename="package://udacity_bot/models/meshes/hokuyo.dae"/>
             </geometry>
+            -->
         </visual>
     </link>
     <joint name="hokuyo_joint" type="fixed">
-        <origin xyz="-0.02 0 0.153" rpy="0 0 0"/>
+        <origin xyz="0.15 0 0.1" rpy="0 0 0"/>
         <parent link="chassis"/>
         <child link="hokuyo"/>

Commit message: changed shell collision and inertias to reflect that of a cylinder

File: urdf/shell.xacro (robot description, xacro)
@@ -9,4 +9,7 @@
  <xacro:macro name="shell_origin">
      <origin xyz="0 0 0" rpy="0 0 -1.5707" />
+ </xacro:macro>
+  <xacro:macro name="cylinder_origin">
+     <origin xyz="0 0 0.05" rpy="0 -1.5707 0" />
  </xacro:macro>
  <xacro:macro name="zero_origin">
@@ -22,4 +25,11 @@
         iyy="0.1" iyz="0"
         izz="0.1"
+      />
+</xacro:macro>
+<xacro:macro name="cylinder_inertia">
+    <inertia
+        ixx="0.2375" ixy="0" ixz="0"
+        iyy="0.075" iyz="0"
+        izz="0.2375"
       />
 </xacro:macro>
@@ -113,17 +123,20 @@
           <mass value="15.0"/>
           <origin xyz="0.0 0 0" rpy=" 0 0 0"/>
-          <xacro:default_inertia/>
+          <!--  <xacro:default_inertia/> -->
+          <xacro:cylinder_inertia/>
     </inertial>
     <collision name='collision'>
-        <xacro:zero_origin/>
-        <geometry>
-            <box size=".4 .2 .1"/>
+        <xacro:cylinder_origin/>
+        <geometry>
+            <!-- <box size=".4 .2 .1"/> -->
+            <cylinder radius="0.1" length="0.4"/>
         </geometry>
     </collision>
     <visual name='chassis_visual'>
-        <!--<xacro:zero_origin/>-->
-        <xacro:shell_origin/>
-        <geometry>
-            <!--<box size=".4 .2 .1"/> -->
+        <xacro:zero_origin/>
+        <!-- <xacro:shell_origin/> -->
+        <geometry>
+            <!--<box size=".4 .2 .1"/>-->
+            <!-- <cylinder radius="0.1" length="0.4"/> -->
             <mesh filename="package://udacity_bot/models/meshes/green_shell.dae"/>
         </geometry>

Commit message: added images of both models

File: urdf/shell.xacro (robot description, xacro)
@@ -134,6 +134,5 @@
     </collision>
     <visual name='chassis_visual'>
-        <xacro:zero_origin/>
-        <!-- <xacro:shell_origin/> -->
+        <xacro:shell_origin/>
         <geometry>
             <!--<box size=".4 .2 .1"/>-->
@@ -245,5 +244,5 @@
     </link>
     <joint name="hokuyo_joint" type="fixed">
-        <origin xyz="0.15 0 0.1" rpy="0 0 0"/>
+        <origin xyz="0.15 0 0.15" rpy="0 0 0"/>
         <parent link="chassis"/>
         <child link="hokuyo"/>
